File: hardware/envlogger2.kicad_sch (KiCad schematic)
At the start: 20 parts, among them J1 Conn_01x06_Pin, J2 Conn_01x03_Socket, J3 Conn_01x03_Socket, SW1 SW_Push, U1 STM32L432KCUx, U2 BME280, Y1 32 kHz

Commit message: Add packet.c and packet.h
Parts:
- added BAT1: BS-7, digikey-footprints:Battery_Holder_Coin_2032_BS-7, symbol dk_Battery-Holders-Clips-Contacts:BS-7
- added C10, C9: 0.1uF, symbol Device:C
Connections:
- net GND: now also U2.1 (GND), U2.5 (SDO), U2.7 (GND), C10.2, C9.2
- net I2C_SCL: now also U2.4 (SCK)
- net I2C_SDA: now also U2.3 (SDI)
- net VDD: now also U2.2 (CSB), U2.6 (VDDIO), U2.8 (VDD), C10.1, C9.1
Other:
- note added: "BME280"
- moved on the sheet: U2
